File: Apple2Card/Apple2Card.kicad_sch (KiCad schematic)
At the start: 77 parts, among them J1 ICSP, J2 Conn_01x25, J3 Conn_01x25, J4 Conn_01x16, J5 SERCON, J6 WIZNET 5500, SW1 SW_Push, U1 ATmega328P-P, U2 74HCT32, U3 74HCT00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

Commit message: Changed pull-down resistor values
Parts:
- R18, R2, R21, R22, R23, R3, R7: value 4k7 -> 10k
Changed lines of the file:
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@@
       (effects (font (size 1.27 1.27)) (justify left))
     )
-    (property "Value" "4k7" (id 1) (at 224.155 158.75 90)
+    (property "Value" "10k" (id 1) (at 224.155 158.75 90)
       (effects (font (size 1.27 1.27)) (justify left))
     )
@@
       (effects (font (size 1.27 1.27)) (justify left))
     )
-    (property "Value" "4k7" (id 1) (at 217.805 158.75 90)
+    (property "Value" "10k" (id 1) (at 217.805 158.75 90)
       (effects (font (size 1.27 1.27)) (justify left))
     )
@@
       (effects (font (size 1.27 1.27)) (justify left))
     )
-    (property "Value" "4k7" (id 1) (at 198.12 158.75 90)
+    (property "Value" "10k" (id 1) (at 198.12 158.75 90)
       (effects (font (size 1.27 1.27)) (justify left))
     )
@@
       (effects (font (size 1.27 1.27)) (justify left))
     )
-    (property "Value" "4k7" (id 1) (at 210.82 158.75 90)
+    (property "Value" "10k" (id 1) (at 210.82 158.75 90)
       (effects (font (size 1.27 1.27)) (justify left))
     )
@@
       (effects (font (size 1.27 1.27)) (justify left))
     )
-    (property "Value" "4k7" (id 1) (at 230.505 158.75 90)
+    (property "Value" "10k" (id 1) (at 230.505 158.75 90)
       (effects (font (size 1.27 1.27)) (justify left))
     )
@@
       (effects (font (size 1.27 1.27)) (justify left))
     )
-    (property "Value" "4k7" (id 1) (at 204.47 158.75 90)
+    (property "Value" "10k" (id 1) (at 204.47 158.75 90)
       (effects (font (size 1.27 1.27)) (justify left))
     )
@@
       (effects (font (size 1.27 1.27)) (justify left))
     )
-    (property "Value" "4k7" (id 1) (at 191.77 158.75 90)
+    (property "Value" "10k" (id 1) (at 191.77 158.75 90)
       (effects (font (size 1.27 1.27)) (justify left))
     )
@@
     )
     (path "/9d68934e-289f-4086-8681-226d8e8ece6c"
-      (reference "R2") (unit 1) (value "4k7") (footprint "Resistor_THT:R_Axial_DIN0207_L6.3mm_D2.5mm_P7.62mm_Horizontal")
+      (reference "R2") (unit 1) (value "10k") (footprint "Resistor_THT:R_Axial_DIN0207_L6.3mm_D2.5mm_P7.62mm_Horizontal")
     )
     (path "/30cf679f-f876-483a-95b7-40e075914504"
-      (reference "R3") (unit 1) (value "4k7") (footprint "Resistor_THT:R_Axial_DIN0207_L6.3mm_D2.5mm_P7.62mm_Horizontal")
+      (reference "R3") (unit 1) (value "10k") (footprint "Resistor_THT:R_Axial_DIN0207_L6.3mm_D2.5mm_P7.62mm_Horizontal")
     )
     (path "/a0cd4d38-f115-45f2-83be-7b9c48e4716b"
@@
     )
     (path "/3cd1b975-dc44-47fb-a883-43bfdfe46373"
-      (reference "R7") (unit 1) (value "4k7") (footprint "Resistor_THT:R_Axial_DIN0207_L6.3mm_D2.5mm_P7.62mm_Horizontal")
+      (reference "R7") (unit 1) (value "10k") (footprint "Resistor_THT:R_Axial_DIN0207_L6.3mm_D2.5mm_P7.62mm_Horizontal")
     )
     (path "/52e3953b-4d68-4321-8211-9cf39a764231"
@@
     )
     (path "/851fb17c-7aa0-4a55-bd2b-57d525ad389f"
-      (reference "R18") (unit 1) (value "4k7") (footprint "Resistor_THT:R_Axial_DIN0207_L6.3mm_D2.5mm_P7.62mm_Horizontal")
+      (reference "R18") (unit 1) (value "10k") (footprint "Resistor_THT:R_Axial_DIN0207_L6.3mm_D2.5mm_P7.62mm_Horizontal")
     )
     (path "/e79fc384-74dc-484b-a360-270761f9e177"
@@
     )
     (path "/26672820-abd4-420c-9526-7367c6ab4ddc"
-      (reference "R21") (unit 1) (value "4k7") (footprint "Resistor_THT:R_Axial_DIN0207_L6.3mm_D2.5mm_P7.62mm_Horizontal")
+      (reference "R21") (unit 1) (value "10k") (footprint "Resistor_THT:R_Axial_DIN0207_L6.3mm_D2.5mm_P7.62mm_Horizontal")
     )
     (path "/00bc57bf-8d06-4b65-a8dd-c5edcb1afa7f"
-      (reference "R22") (unit 1) (value "4k7") (footprint "Resistor_THT:R_Axial_DIN0207_L6.3mm_D2.5mm_P7.62mm_Horizontal")
+      (reference "R22") (unit 1) (value "10k") (footprint "Resistor_THT:R_Axial_DIN0207_L6.3mm_D2.5mm_P7.62mm_Horizontal")
     )
     (path "/6d20c98b-f235-4d8e-8a08-56fd3d5c6886"
-      (reference "R23") (unit 1) (value "4k7") (footprint "Resistor_THT:R_Axial_DIN0207_L6.3mm_D2.5mm_P7.62mm_Horizontal")
+      (reference "R23") (unit 1) (value "10k") (footprint "Resistor_THT:R_Axial_DIN0207_L6.3mm_D2.5mm_P7.62mm_Horizontal")
     )
     (path "/59cbc428-c63f-4e29-be89-d9e971907c8a"
